Commit message: fix(session_6): resolve platform startup errors, missing wheels, and RViz configs in tb3_sensor_lab

File: session_6/tb3_sensor_lab/urdf/waffle.urdf (robot description, URDF)
Before this commit: robot waffle, 7 links, 6 joints
Links:
- added link caster_back_left_link
- added link caster_back_right_link
- added link wheel_left_link; visual cylinder length=0.018 radius=0.033
- added link wheel_right_link; visual cylinder length=0.018 radius=0.033
- link base_link: geometry visual box size=0.265 0.265 0.089
Joints:
- added joint caster_back_left_joint: type fixed, parent base_link, child caster_back_left_link, origin xyz=-0.177 0.064 -0.005 rpy=0 0 0
- added joint caster_back_right_joint: type fixed, parent base_link, child caster_back_right_link, origin xyz=-0.177 -0.064 -0.005 rpy=0 0 0
- added joint wheel_left_joint: type continuous, parent base_link, child wheel_left_link, origin xyz=0 0.144 0.023 rpy=-1.5708 0 0, axis 0 0 1
- added joint wheel_right_joint: type continuous, parent base_link, child wheel_right_link, origin xyz=0 -0.144 0.023 rpy=-1.5708 0 0, axis 0 0 1
- joint camera_rgb_optical_joint: origin xyz=0 0 0 rpy=-1.57 0 -1.57 -> xyz=0 0 0 rpy=-1.5708 0 -1.5708
- joint imu_joint: origin xyz=0.0 0 0.068 rpy=0 0 0 -> xyz=0 0 0.068 rpy=0 0 0
