Commit message: feat(description): add 3D visual models for chassis, wheels, roll cage, and sensor enclosures; set rviz fixed frame to base_link

File: ev_description/urdf/ev_buggy.urdf.xacro (robot description, xacro)
@@ -5,6 +5,131 @@
   <!-- base_link: Rear axle center projected down to the ground plane       -->
   <!-- ===================================================================== -->
-  <link name="base_link"/>
-  <!-- Include rigid sensor mount transforms -->
+  <link name="base_link">
+    <visual>
+      <origin xyz="0.65 0 0.02" rpy="0 0 0"/>
+      <geometry>
+        <box size="0.1 0.1 0.02"/>
+      </geometry>
+      <material name="origin_marker">
+        <color rgba="1.0 0.84 0.0 0.8"/>
+      </material>
+    </visual>
+  </link>
+  <!-- ===================================================================== -->
+  <!-- MAIN CHASSIS BODY                                                     -->
+  <!-- ===================================================================== -->
+  <link name="chassis_link">
+    <!-- Main lower hull / belly pan -->
+    <visual>
+      <origin xyz="0.65 0.0 0.18" rpy="0 0 0"/>
+      <geometry>
+        <box size="1.50 0.70 0.16"/>
+      </geometry>
+      <material name="chassis_dark">
+        <color rgba="0.15 0.16 0.18 1.0"/>
+      </material>
+    </visual>
+    <!-- Upper body cowl / hood -->
+    <visual>
+      <origin xyz="0.95 0.0 0.30" rpy="0 0.08 0"/>
+      <geometry>
+        <box size="0.75 0.65 0.10"/>
+      </geometry>
+      <material name="body_paint">
+        <color rgba="0.12 0.53 0.90 1.0"/>
+      </material>
+    </visual>
+    <!-- Cockpit / Roll cage arch -->
+    <visual>
+      <origin xyz="0.45 0.0 0.55" rpy="0 0 0"/>
+      <geometry>
+        <box size="0.70 0.62 0.50"/>
+      </geometry>
+      <material name="roll_cage">
+        <color rgba="0.25 0.25 0.28 0.6"/>
+      </material>
+    </visual>
+    <!-- Roll cage top roof plate (Sensor mounting platform) -->
+    <visual>
+      <origin xyz="0.45 0.0 0.80" rpy="0 0 0"/>
+      <geometry>
+        <box size="0.60 0.58 0.02"/>
+      </geometry>
+      <material name="roof_plate">
+        <color rgba="0.18 0.18 0.20 1.0"/>
+      </material>
+    </visual>
+  </link>
+  <joint name="chassis_joint" type="fixed">
+    <parent link="base_link"/>
+    <child link="chassis_link"/>
+    <origin xyz="0.0 0.0 0.0" rpy="0 0 0"/>
+  </joint>
+  <!-- ===================================================================== -->
+  <!-- WHEELS (Visual representation of 4-wheel EV platform)                 -->
+  <!-- ===================================================================== -->
+  <!-- Rear Left Wheel -->
+  <link name="rear_left_wheel">
+    <visual>
+      <origin xyz="0 0 0" rpy="1.570796 0 0"/>
+      <geometry>
+        <cylinder radius="0.18" length="0.12"/>
+      </geometry>
+      <material name="tire_rubber">
+        <color rgba="0.08 0.08 0.08 1.0"/>
+      </material>
+    </visual>
+  </link>
+  <joint name="rear_left_wheel_joint" type="fixed">
+    <parent link="base_link"/>
+    <child link="rear_left_wheel"/>
+    <origin xyz="0.0 0.40 0.18" rpy="0 0 0"/>
+  </joint>
+  <!-- Rear Right Wheel -->
+  <link name="rear_right_wheel">
+    <visual>
+      <origin xyz="0 0 0" rpy="1.570796 0 0"/>
+      <geometry>
+        <cylinder radius="0.18" length="0.12"/>
+      </geometry>
+      <material name="tire_rubber"/>
+    </visual>
+  </link>
+  <joint name="rear_right_wheel_joint" type="fixed">
+    <parent link="base_link"/>
+    <child link="rear_right_wheel"/>
+    <origin xyz="0.0 -0.40 0.18" rpy="0 0 0"/>
+  </joint>
+  <!-- Front Left Wheel -->
+  <link name="front_left_wheel">
+    <visual>
+      <origin xyz="0 0 0" rpy="1.570796 0 0"/>
+      <geometry>
+        <cylinder radius="0.18" length="0.12"/>
+      </geometry>
+      <material name="tire_rubber"/>
+    </visual>
+  </link>
+  <joint name="front_left_wheel_joint" type="fixed">
+    <parent link="base_link"/>
+    <child link="front_left_wheel"/>
+    <origin xyz="1.30 0.40 0.18" rpy="0 0 0"/>
+  </joint>
+  <!-- Front Right Wheel -->
+  <link name="front_right_wheel">
+    <visual>
+      <origin xyz="0 0 0" rpy="1.570796 0 0"/>
+      <geometry>
+        <cylinder radius="0.18" length="0.12"/>
+      </geometry>
+      <material name="tire_rubber"/>
+    </visual>
+  </link>
+  <joint name="front_right_wheel_joint" type="fixed">
+    <parent link="base_link"/>
+    <child link="front_right_wheel"/>
+    <origin xyz="1.30 -0.40 0.18" rpy="0 0 0"/>
+  </joint>
+  <!-- Include rigid sensor mount transforms and 3D visual models -->
   <xacro:include filename="$(find ev_description)/urdf/sensor_mounts.xacro"/>
 </robot>

File: ev_description/urdf/sensor_mounts.xacro (robot description, xacro)
@@ -4,5 +4,26 @@
   <!-- 1. 2D PLANAR LiDAR: Slamtec RPLIDAR S3 (Overhead roll arch plate)     -->
   <!-- ===================================================================== -->
-  <link name="laser_frame"/>
+  <link name="laser_frame">
+    <visual>
+      <!-- LiDAR base puck -->
+      <origin xyz="0 0 -0.015" rpy="0 0 0"/>
+      <geometry>
+        <cylinder radius="0.038" length="0.035"/>
+      </geometry>
+      <material name="lidar_black">
+        <color rgba="0.1 0.1 0.1 1.0"/>
+      </material>
+    </visual>
+    <visual>
+      <!-- LiDAR optic window ring -->
+      <origin xyz="0 0 0.005" rpy="0 0 0"/>
+      <geometry>
+        <cylinder radius="0.035" length="0.015"/>
+      </geometry>
+      <material name="lidar_optical_ring">
+        <color rgba="0.0 0.95 0.85 0.9"/>
+      </material>
+    </visual>
+  </link>
   <joint name="laser_joint" type="fixed">
     <parent link="base_link"/>
@@ -13,5 +34,26 @@
   <!-- 2. INERTIAL MEASUREMENT UNIT: WitMotion WT901 (Center spine / CG)     -->
   <!-- ===================================================================== -->
-  <link name="imu_link"/>
+  <link name="imu_link">
+    <visual>
+      <!-- Anodized aluminum IMU enclosure -->
+      <origin xyz="0 0 0" rpy="0 0 0"/>
+      <geometry>
+        <box size="0.052 0.038 0.016"/>
+      </geometry>
+      <material name="imu_blue">
+        <color rgba="0.1 0.45 0.95 1.0"/>
+      </material>
+    </visual>
+    <visual>
+      <!-- Status LED / Pin header accent -->
+      <origin xyz="0.02 0 0.009" rpy="0 0 0"/>
+      <geometry>
+        <box size="0.008 0.008 0.003"/>
+      </geometry>
+      <material name="imu_led">
+        <color rgba="0.2 1.0 0.2 1.0"/>
+      </material>
+    </visual>
+  </link>
   <joint name="imu_joint" type="fixed">
     <parent link="base_link"/>
@@ -22,5 +64,36 @@
   <!-- 3. GNSS RECEIVER: Holybro Pixhawk M9N (Elevated rear mast)            -->
   <!-- ===================================================================== -->
-  <link name="gps_link"/>
+  <link name="gps_link">
+    <visual>
+      <!-- Mast pole -->
+      <origin xyz="0 0 -0.25" rpy="0 0 0"/>
+      <geometry>
+        <cylinder radius="0.006" length="0.50"/>
+      </geometry>
+      <material name="carbon_mast">
+        <color rgba="0.15 0.15 0.15 1.0"/>
+      </material>
+    </visual>
+    <visual>
+      <!-- GPS dome puck antenna -->
+      <origin xyz="0 0 0" rpy="0 0 0"/>
+      <geometry>
+        <cylinder radius="0.032" length="0.016"/>
+      </geometry>
+      <material name="gps_white">
+        <color rgba="0.95 0.95 0.95 1.0"/>
+      </material>
+    </visual>
+    <visual>
+      <!-- Direction arrow mark -->
+      <origin xyz="0.012 0 0.009" rpy="0 0 0"/>
+      <geometry>
+        <box size="0.015 0.005 0.002"/>
+      </geometry>
+      <material name="gps_red">
+        <color rgba="0.9 0.1 0.1 1.0"/>
+      </material>
+    </visual>
+  </link>
   <joint name="gps_joint" type="fixed">
     <parent link="base_link"/>
@@ -31,5 +104,34 @@
   <!-- 4. STEREO DEPTH CAMERA: Stereolabs ZED 2i (Front impact cowl bracket) -->
   <!-- ===================================================================== -->
-  <link name="camera_link"/>
+  <link name="camera_link">
+    <visual>
+      <!-- Main camera bar body -->
+      <origin xyz="0 0 0" rpy="0 0 0"/>
+      <geometry>
+        <box size="0.035 0.175 0.030"/>
+      </geometry>
+      <material name="zed_body">
+        <color rgba="0.12 0.12 0.12 1.0"/>
+      </material>
+    </visual>
+    <!-- Left optical lens -->
+    <visual>
+      <origin xyz="0.018 0.06 0" rpy="0 1.570796 0"/>
+      <geometry>
+        <cylinder radius="0.011" length="0.004"/>
+      </geometry>
+      <material name="zed_lens">
+        <color rgba="0.1 0.2 0.4 1.0"/>
+      </material>
+    </visual>
+    <!-- Right optical lens -->
+    <visual>
+      <origin xyz="0.018 -0.06 0" rpy="0 1.570796 0"/>
+      <geometry>
+        <cylinder radius="0.011" length="0.004"/>
+      </geometry>
+      <material name="zed_lens"/>
+    </visual>
+  </link>
   <joint name="camera_joint" type="fixed">
     <parent link="base_link"/>
