Commit message: feat(stage4): bring up Stereolabs ZED 2i depth camera driver, HD720@15FPS config, and RViz pointcloud layout

File: ev_description/urdf/sensor_mounts.xacro (robot description, xacro)
@@ -37,4 +37,11 @@
     <origin xyz="1.25 0.00 0.35" rpy="0.0 0.0 0.0"/>
   </joint>
+  <!-- Bridge to ZED wrapper base link -->
+  <link name="zed_camera_link"/>
+  <joint name="zed_camera_joint" type="fixed">
+    <parent link="camera_link"/>
+    <child link="zed_camera_link"/>
+    <origin xyz="0.00 0.00 0.00" rpy="0.0 0.0 0.0"/>
+  </joint>
   <!-- ===================================================================== -->
   <!-- 5. OPTICAL AXIS SUB-LINK (Standard Computer Vision: Z-forward, X-right)-->

Commit message: feat(student): prepare ev_ws student work branch for 3-team parallel lab and phase 1 bringup

File: ev_description/urdf/sensor_mounts.xacro (robot description, xacro)
@@ -29,5 +29,5 @@
     <parent link="base_link"/>
     <child link="laser_frame"/>
-    <origin xyz="1.20 0.00 0.45" rpy="0.0 0.0 0.0"/>
+    <origin xyz="0.0 0.0 0.0" rpy="0.0 0.0 0.0"/>
   </joint>
   <!-- ===================================================================== -->
@@ -59,5 +59,5 @@
     <parent link="base_link"/>
     <child link="imu_link"/>
-    <origin xyz="0.40 0.00 0.25" rpy="0.0 0.0 0.0"/>
+    <origin xyz="0.0 0.0 0.0" rpy="0.0 0.0 0.0"/>
   </joint>
   <!-- ===================================================================== -->
@@ -99,5 +99,5 @@
     <parent link="base_link"/>
     <child link="gps_link"/>
-    <origin xyz="0.10 0.00 1.10" rpy="0.0 0.0 0.0"/>
+    <origin xyz="0.0 0.0 0.0" rpy="0.0 0.0 0.0"/>
   </joint>
   <!-- ===================================================================== -->
@@ -137,5 +137,5 @@
     <parent link="base_link"/>
     <child link="camera_link"/>
-    <origin xyz="1.25 0.00 0.35" rpy="0.0 0.0 0.0"/>
+    <origin xyz="0.0 0.0 0.0" rpy="0.0 0.0 0.0"/>
   </joint>
   <!-- Bridge to ZED wrapper base link -->
@@ -153,5 +153,5 @@
     <parent link="camera_link"/>
     <child link="camera_depth_optical_frame"/>
-    <origin xyz="0.00 0.00 0.00" rpy="-1.5708 0.0 -1.5708"/>
+    <origin xyz="0.00 0.00 0.00" rpy="0.0 0.0 0.0"/>
   </joint>
 </robot>

Commit message: Update sensor_mounts.xacro
updated gps mount center physical measurements - Huda and Amal

File: ev_description/urdf/sensor_mounts.xacro (robot description, xacro)
@@ -99,5 +99,5 @@
     <parent link="base_link"/>
     <child link="gps_link"/>
-    <origin xyz="0.10 0.00 1.10" rpy="0.0 0.0 0.0"/>
+    <origin xyz="-90 0.00 98" rpy="0.0 0.0 0.0"/>
   </joint>
   <!-- ===================================================================== -->

Commit message: Update laser_joint origin coordinates

File: ev_description/urdf/sensor_mounts.xacro (robot description, xacro)
@@ -29,5 +29,5 @@
     <parent link="base_link"/>
     <child link="laser_frame"/>
-    <origin xyz="1.20 0.00 0.45" rpy="0.0 0.0 0.0"/>
+    <origin xyz="-77.00 0.00 95.00" rpy="0.0 0.0 0.0"/>
   </joint>
   <!-- ===================================================================== -->

Commit message: Update sensor_mounts.xacro
Update camera position

File: ev_description/urdf/sensor_mounts.xacro (robot description, xacro)
@@ -29,5 +29,5 @@
     <parent link="base_link"/>
     <child link="laser_frame"/>
-    <origin xyz="-77.00 0.00 95.00" rpy="0.0 0.0 0.0"/>
+    <origin xyz="1.20 0.00 0.45" rpy="0.0 0.0 0.0"/>
   </joint>
   <!-- ===================================================================== -->
@@ -137,5 +137,5 @@
     <parent link="base_link"/>
     <child link="camera_link"/>
-    <origin xyz="1.25 0.00 0.35" rpy="0.0 0.0 0.0"/>
+    <origin xyz="0.36 0.00 0.67" rpy="0.0 0.0 0.0"/>
   </joint>
   <!-- Bridge to ZED wrapper base link -->

Commit message: Update sensor_mounts.xacro
updating measurements for gps from cm to meter

File: ev_description/urdf/sensor_mounts.xacro (robot description, xacro)
@@ -99,5 +99,5 @@
     <parent link="base_link"/>
     <child link="gps_link"/>
-    <origin xyz="-90 0.00 98" rpy="0.0 0.0 0.0"/>
+    <origin xyz="-0.90 0.00 0.98" rpy="0.0 0.0 0.0"/>
   </joint>
   <!-- ===================================================================== -->

Commit message: Fix laser_joint origin coordinates

File: ev_description/urdf/sensor_mounts.xacro (robot description, xacro)
@@ -29,5 +29,5 @@
     <parent link="base_link"/>
     <child link="laser_frame"/>
-    <origin xyz="-77.00 0.00 95.00" rpy="0.0 0.0 0.0"/>
+    <origin xyz="-0.77 0.00 0.95" rpy="0.0 0.0 0.0"/>
   </joint>
   <!-- ===================================================================== -->

Commit message: Update IMU joint origin position

File: ev_description/urdf/sensor_mounts.xacro (robot description, xacro)
@@ -59,5 +59,5 @@
     <parent link="base_link"/>
     <child link="imu_link"/>
-    <origin xyz="0.0 0.0 0.0" rpy="0.0 0.0 0.0"/>
+    <origin xyz="-150 0.0 59" rpy="0.0 0.0 0.0"/>
   </joint>
   <!-- ===================================================================== -->
